File: Breakout/Dual Vertical/Dual Vertical Breakout Module.brd (EAGLE design)
At the start: 25.4 x 30.5 mm, 4 parts

Commit message: Updated Root1 connector labels. Renamed Dual Horizontal Breakout Module. Both breakout files need silkscreen.
Signed-off-by: Cruz Monrreal II <Cruz.Monrreal@gmail.com>
Connections:
- net 01 renamed TXO
- net 02 renamed RXI
Changed lines of the file:
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@@
 <wire x1="7.62" y1="20.955" x2="8.255" y2="20.32" width="0.3048" layer="16"/>
 </signal>
-<signal name="01">
+<signal name="TXO">
 <contactref element="U$8" pad="01@VIA"/>
 <contactref element="U$8" pad="01@1"/>
@@
 <wire x1="8.89" y1="20.32" x2="13.335" y2="15.875" width="0.3048" layer="1"/>
 </signal>
-<signal name="02">
+<signal name="RXI">
 <contactref element="U$8" pad="02@VIA"/>
 <contactref element="U$8" pad="02@1"/>
