File: uC/LPC/1343/LPC1343 Module.sch (EAGLE design)
At the start: 36 parts, among them CN1 USBMINIB, Q1 MMBT2907A, U1 LPC1343FBD48, U3 MCP130T, X1 USB-MICROB, Y2 12MHz

Commit message: Updated Root1 header on LPC1343 MOdule
Signed-off-by: Cruz Monrreal II <Cruz.Monrreal@gmail.com>
Parts:
- removed U$9: DF40.30PIN.RECEPTACLE, hirose:DF40.30PIN.RECEPTACLE
Other:
- note removed: "!RST"
- note removed: "3.3V"
- note removed: "DF40.12"
- note removed: "GND"
- note removed: "IO.0/TDI"
- note removed: "IO.1/!TRST"
- note removed: "IO.2"
- note removed: "IO.3"
- note removed: "RxI"
- note removed: "SWCLK/TCK"
- note removed: "SWDIO/TMS"
- note removed: "SWO/TDO"
- note removed: "TxO"
Changed lines of the file:
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@@
 <?xml version="1.0" encoding="utf-8"?>
 <!DOCTYPE eagle SYSTEM "eagle.dtd">
-<eagle version="6.1">
+<eagle version="6.3">
 <drawing>
 <settings>
@@
 <layers>
 <layer number="1" name="Top" color="4" fill="1" visible="no" active="no"/>
+<layer number="2" name="Route2" color="1" fill="3" visible="no" active="no"/>
+<layer number="3" name="Route3" color="4" fill="3" visible="no" active="no"/>
+<layer number="4" name="Route4" color="1" fill="4" visible="no" active="no"/>
+<layer number="5" name="Route5" color="4" fill="4" visible="no" active="no"/>
+<layer number="6" name="Route6" color="1" fill="8" visible="no" active="no"/>
+<layer number="7" name="Route7" color="4" fill="8" visible="no" active="no"/>
+<layer number="8" name="Route8" color="1" fill="2" visible="no" active="no"/>
+<layer number="9" name="Route9" color="4" fill="2" visible="no" active="no"/>
+<layer number="10" name="Route10" color="1" fill="7" visible="no" active="no"/>
+<layer number="11" name="Route11" color="4" fill="7" visible="no" active="no"/>
+<layer number="12" name="Route12" color="1" fill="5" visible="no" active="no"/>
+<layer number="13" name="Route13" color="4" fill="5" visible="no" active="no"/>
+<layer number="14" name="Route14" color="1" fill="6" visible="no" active="no"/>
+<layer number="15" name="Route15" color="4" fill="6" visible="no" active="no"/>
 <layer number="16" name="Bottom" color="1" fill="1" visible="no" active="no"/>
 <layer number="17" name="Pads" color="2" fill="1" visible="no" active="no"/>
@@
 <part name="U$38" library="microbuilder" deviceset="GND" device=""/>
 <part name="R6" library="microbuilder" deviceset="RESISTOR" device="0603" value="1K"/>
-<part name="U$9" library="hirose" deviceset="DF40.30PIN" device=".RECEPTACLE"/>
 <part name="X1" library="SparkFun" deviceset="USB" device="-MICROB"/>
 </parts>
@@
 <text x="276.86" y="162.56" size="1.778" layer="97">R7 + R14 will cause bootloader to boot into USB/MSC mode if USB</text>
 <text x="276.86" y="160.02" size="1.778" layer="97">is connected (0.3 HIGH), otherwise it will use UART/ISP (0.3 LOW)</text>
-<text x="55.88" y="104.14" size="1.778" layer="97">DF40.12</text>
-<text x="60.96" y="99.06" size="1.778" layer="97" rot="MR0">SWCLK/TCK</text>
-<text x="60.96" y="96.52" size="1.778" layer="97" rot="MR0">SWDIO/TMS</text>
-<text x="63.5" y="99.06" size="1.778" layer="97">SWO/TDO</text>
-<text x="63.5" y="96.52" size="1.778" layer="97">IO.0/TDI</text>
-<text x="63.5" y="93.98" size="1.778" layer="97">IO.1/!TRST</text>
-<text x="60.96" y="86.36" size="1.778" layer="97" rot="MR0">GND</text>
-<text x="63.5" y="86.36" size="1.778" layer="97">3.3V</text>
-<text x="60.96" y="93.98" size="1.778" layer="97" rot="MR0">TxO</text>
-<text x="60.96" y="91.44" size="1.778" layer="97" rot="MR0">RxI</text>
-<text x="60.96" y="88.9" size="1.778" layer="97" rot="MR0">!RST</text>
-<text x="63.5" y="91.44" size="1.778" layer="97">IO.2</text>
-<text x="63.5" y="88.9" size="1.778" layer="97">IO.3</text>
 </plain>
 <instances>
@@
 <instance part="U$38" gate="G$1" x="317.5" y="185.42"/>
 <instance part="R6" gate="G$1" x="325.12" y="203.2"/>
-<instance part="U$9" gate="U" x="106.68" y="109.22"/>
 <instance part="X1" gate="G$1" x="264.16" y="129.54"/>
 </instances>
@@
 <pinref part="U$5" gate="G$1" pin="GND"/>
 <pinref part="U$8" gate="G$2" pin="GND"/>
-<wire x1="203.2" y1="124.46" x2="205.74" y2="127" width="0.1524" layer="91"/>
-<junction x="205.74" y="127"/>
+<wire x1="203.2" y1="124.46" x2="210.82" y2="127" width="0.1524" layer="91"/>
+<junction x="210.82" y="127"/>
 </segment>
 <segment>
@@
 <pinref part="U$8" gate="G$2" pin="3.3V"/>
 <pinref part="U$6" gate="G$1" pin="3.3V"/>
-<wire x1="205.74" y1="129.54" x2="203.2" y2="132.08" width="0.1524" layer="91"/>
-<junction x="205.74" y="129.54"/>
+<wire x1="210.82" y1="129.54" x2="203.2" y2="132.08" width="0.1524" layer="91"/>
+<junction x="210.82" y="129.54"/>
 </segment>
 <segment>
@@
 <segment>
 <pinref part="U$8" gate="G$1" pin="01"/>
-<junction x="175.26" y="111.76"/>
+<junction x="175.26" y="106.68"/>
 </segment>
 </net>
@@
 <segment>
 <pinref part="U$8" gate="G$1" pin="02"/>
-<junction x="175.26" y="109.22"/>
+<junction x="175.26" y="104.14"/>
 </segment>
 </net>
@@
 <segment>
 <pinref part="U$8" gate="G$1" pin="03"/>
-<junction x="175.26" y="106.68"/>
+<junction x="175.26" y="101.6"/>
 </segment>
 </net>
@@
 <segment>
 <pinref part="U$8" gate="G$1" pin="04"/>
-<junction x="175.26" y="104.14"/>
+<junction x="175.26" y="99.06"/>
 </segment>
 </net>
@@
 <segment>
 <pinref part="U$8" gate="G$1" pin="05"/>
-<junction x="175.26" y="101.6"/>
+<junction x="175.26" y="96.52"/>
 </segment>
 </net>
@@
 <segment>
 <pinref part="U$8" gate="G$1" pin="06"/>
-<junction x="175.26" y="99.06"/>
+<junction x="175.26" y="93.98"/>
 </segment>
 </net>
@@
 <segment>
 <pinref part="U$8" gate="G$1" pin="07"/>
-<junction x="175.26" y="96.52"/>
+<junction x="175.26" y="91.44"/>
 </segment>
 </net>
@@
 <segment>
 <pinref part="U$8" gate="G$1" pin="WAKE"/>
-<junction x="175.26" y="93.98"/>
-<wire x1="175.26" y1="93.98" x2="182.88" y2="93.98" width="0.1524" layer="91"/>
+<junction x="175.26" y="88.9"/>
+<wire x1="175.26" y1="88.9" x2="182.88" y2="93.98" width="0.1524" layer="91"/>
 <label x="182.88" y="93.98" size="1.27" layer="95"/>
 </segment>
