File: IO/Debug/Debug Module.brd (EAGLE design)
At the start: 25.4 x 25.4 mm, 25 parts, among them U1 74HC541, U2 74HC541

Commit message: Completed Debug Module Added/began Thermocouple Module
Signed-off-by: Cruz Monrreal II <Cruz.Monrreal@gmail.com>
Routing:
- net 3.3V: track 3.65 -> 30.3 mm, vias 0 -> 2
- net RST: track 0.00 -> 24.0 mm, vias 0 -> 1
- net SDA: track 0.00 -> 8.56 mm, vias 0 -> 1
- net MISO: track 0.00 -> 8.44 mm, vias 0 -> 1
- net RXI: track 0.00 -> 8.31 mm, vias 0 -> 1
- net SCL: track 0.00 -> 8.23 mm
- net SCLK: track 0.00 -> 8.11 mm
- net MOSI: track 0.00 -> 6.31 mm
- net TXO: track 0.00 -> 5.58 mm
- net GND: track 2.30 -> 4.61 mm, vias 2 -> 6
- net 02: track 11.1 -> 9.50 mm, vias 1 -> 0
- net 06: track 7.88 -> 6.43 mm
- net 03: track 12.1 -> 11.6 mm, vias 0 -> 1
- net 04: track 11.2 -> 10.9 mm, vias 1 -> 0
